Commit message: !UNTESTED! Implement IK calculation

File: dev_ws/robot/urdf/robot.urdf (robot description, URDF)
Before this commit: robot example_robot, 5 links, 4 joints
Links:
- added link ee_pitch, mass 0.0
- added link ee_yaw, mass 0.0
Joints:
- removed joint ee_joint
- added joint ee_pitch_joint: type revolute, parent ee_yaw, child ee_pitch, origin xyz=0 0 0 rpy=0 0 0, axis 0 1 0, limit lower=-3.14 upper=3.14 effort=10 velocity=2
- added joint ee_roll_joint: type revolute, parent ee_pitch, child ee, origin xyz=0 0 0 rpy=0 0 0, axis 1 0 0, limit lower=-3.14 upper=3.14 effort=10 velocity=2
- added joint ee_yaw_joint: type revolute, parent link3, child ee_yaw, origin xyz=0.5 0 0 rpy=0 0 0, axis 0 0 1, limit lower=-3.14 upper=3.14 effort=10 velocity=2
- joint q3: origin xyz=0 0 0.5 rpy=0 0 0 -> xyz=0.5 0 0 rpy=0 0 0
