Commit message: Fake balljoint to allow IK to find a solution

File: dev_ws/robot/urdf/robot_w_balljoint.urdf (robot description, URDF)
Before this commit: robot example_robot, 6 links, 5 joints
Links:
- added link ee_pitch
- added link ee_yaw
Joints:
- removed joint ee_joint
- added joint ee_pitch_joint: type revolute, parent ee_yaw, child ee_pitch, origin xyz=0 0 0 rpy=0 0 0, axis 0 1 0, limit lower=-3.14 upper=3.14 effort=10 velocity=2
- added joint ee_roll_joint: type revolute, parent ee_pitch, child ee, origin xyz=0 0 0 rpy=0 0 0, axis 1 0 0, limit lower=-3.14 upper=3.14 effort=10 velocity=2
- added joint ee_yaw_joint: type revolute, parent link3, child ee_yaw, origin xyz=5 0 0 rpy=0 0 0, axis 0 0 1, limit lower=-3.14 upper=3.14 effort=10 velocity=2
